File: Nemesis/DRV8874.kicad_sch (KiCad schematic)
At the start: 1 part, among them U2 DRV8874PWPR

Commit message: Add files via upload
Parts:
- added C1: 22nF, symbol Device:C
- added C2: 220nF, symbol Device:C
- added C3, C4: 4.7nF, symbol Device:C
- added C5, C6: 0.1nF, symbol Device:C
- added D1: D_Zener, symbol Device:D_Zener
- added Q1: Q_PMOS, symbol Device:Q_PMOS
- added R10: 10k, symbol Device:R
- added R11: NP, symbol Device:R
- added R12: 100k, symbol Device:R
- added R8: 2.49k, symbol Device:R
- added R9: 20k, symbol Device:R
Connections:
- net CS: now also U2.6 (IPROPI), R8.1
- net FLT: now also U2.4 (NFAULT)
- net GND: now also U2.15 (GND), U2.9 (PGND), C3.1, C4.1, C5.1, C6.1, R11.2, R12.2, R8.2, R9.2
- net IMODE: now also U2.7 (IMODE), R9.1
- net IN1 EN: now also U2.1 (EN/IN1)
- net IN2 PH: now also U2.2 (PH/IN2)
- net OUT1: now also U2.8 (OUT1)
- net OUT2: now also U2.10 (OUT2)
- net PMODE: now also U2.16 (PMODE)
- net SLP: now also U2.3 (NSLEEP), R10.1
- net VIN: now also C3.2, C4.2, C5.2, C6.2, D1.1 (K), Q1.S
- net VM: now also U2.11 (VM), C2.2, Q1.D
- net VREF: now also U2.5 (VREF), R10.2, R11.1
- net at U2.12 (VCP): now also C2.1
- net at U2.13 (CPH): now also C1.1
- net at U2.14 (CPL): now also C1.2
- new net: D1.2 (A), Q1.G, R12.1
Other:
- moved on the sheet: U2

Commit message: Add files via upload
Parts:
- removed C3: 4.7nF, symbol Device:C
- removed C5: 0.1nF, symbol Device:C
- added C10: 4.7nF, Capacitor_SMD:C_0805_2012Metric_Pad1.18x1.45mm_HandSolder, symbol Device:C
- added C12: 0.1nF, Capacitor_SMD:C_0805_2012Metric_Pad1.18x1.45mm_HandSolder, symbol Device:C
- C11: renamed from C4; footprint (none) -> Capacitor_SMD:C_0805_2012Metric_Pad1.18x1.45mm_HandSolder
- C13: renamed from C6; footprint (none) -> Capacitor_SMD:C_0805_2012Metric_Pad1.18x1.45mm_HandSolder
- C14: renamed from C1; footprint (none) -> Capacitor_SMD:C_0805_2012Metric_Pad1.18x1.45mm_HandSolder
- C9: renamed from C2; footprint (none) -> Capacitor_SMD:C_0805_2012Metric_Pad1.18x1.45mm_HandSolder
- D1: value D_Zener -> 16.2V; footprint (none) -> Diode_SMD:D_SOD-323_HandSoldering
- Q1: footprint (none) -> Package_TO_SOT_SMD:TO-252-2
- R10: renamed from R9; footprint (none) -> Resistor_SMD:R_0805_2012Metric_Pad1.20x1.40mm_HandSolder
- R11: renamed from R10; footprint (none) -> Resistor_SMD:R_0805_2012Metric_Pad1.20x1.40mm_HandSolder
- R12: renamed from R11; footprint (none) -> Resistor_SMD:R_0805_2012Metric_Pad1.20x1.40mm_HandSolder
- R13: renamed from R12; footprint (none) -> Resistor_SMD:R_0805_2012Metric_Pad1.20x1.40mm_HandSolder
- R14: renamed from R8; footprint (none) -> Resistor_SMD:R_0805_2012Metric_Pad1.20x1.40mm_HandSolder
Connections:
- net GND: now also C10.1, C12.1
- net VIN: now also C10.2, C12.2
- no-connect marks 0 -> 1
