File: Nemesis/LSM6DSO.kicad_sch (KiCad schematic)
At the start: 8 parts, among them U3 LSM6DSO

Commit message: Add files via upload
Parts:
- added C1: 1.0 uF, Capacitor_SMD:C_0805_2012Metric, symbol Device:C
- added C2, C6, C7: 0.1 uF, Capacitor_SMD:C_0805_2012Metric, symbol Device:C
- added C3, C4: 4.7 uF, Capacitor_SMD:C_0805_2012Metric, symbol Device:C
- added C5: 1 uF, Capacitor_SMD:C_0805_2012Metric, symbol Device:C
- added R8, R9: 10k, Resistor_SMD:R_0805_2012Metric, symbol Device:R
- R1, R2, R3, R4, R5, R6, R7: footprint (none) -> Resistor_SMD:R_0805_2012Metric
Connections:
- net CS: now also R6.1; no longer R4.2
- net GND: now also C1.2, C2.2, C3.2, C4.2, C5.2, C6.2, C7.2
- net OCS Aux: now also R9.1; no longer R7.1
- net SCL: now also R4.1
- net SCx: now also R8.1; no longer R6.1
- net SDA: now also R3.1
- net SDO: now also R5.1; no longer R3.2
- net SDx: now also R7.1; no longer R5.1
- net VIN: now also R3.2, R4.2, C1.1, C2.1, C3.1, C4.1, C5.1, C6.1, C7.1, R8.2, R9.2; no longer R3.1, R4.1
- net SDO Aux renamed SDO AUX
- no-connect marks 0 -> 3
Other:
- company: (none) -> Cal Poly
- title: (none) -> Accelerometer and Gyrometer
