File: Nemesis/Nemesis.kicad_sch (KiCad schematic)
At the start: 6 parts, among them J1 Screw_Terminal_01x02, U1 NODEMCU-32S

Commit message: Add files via upload
Parts:
- added J2, J3: Screw_Terminal_01x02, TerminalBlock_Phoenix:TerminalBlock_Phoenix_MKDS-1,5-2-5.08_1x02_P5.08mm_Horizontal, symbol Connector:Screw_Terminal_01x02
Connections:
- net +3V3: now reaches U1.J1_1 (3.3V)
- net GPIO27: now reaches U1.J1_11 (IO27)
- net GPIO14: now reaches U1.J1_12 (IO14)
- net GND: now reaches U1.J1_14 (GND), U1.J2_1 (GND), U1.J2_7 (GND)
- net GND: now also J1.2 (Pin_2)
- net DRV8874/IN1 EN: now reaches U1.J2_11 (IO17)
- net DRV8874/IN2 PH: now reaches U1.J2_12 (IO16)
- net VMOT: now reaches J1.1 (Pin_1)
- new net DRV8874/OUT1: J2.1 (Pin_1)
- new net DRV8874/OUT2: J2.2 (Pin_2)
- new net DRV8875/OUT1: J3.1 (Pin_1)
- new net DRV8875/OUT2: J3.2 (Pin_2)
- no-connect marks 0 -> 22
Other:
- added sheet DRV8875 (DRV8874.kicad_sch)
- sheet DRV8874 ports: added GND, IN1 EN, IN2 PH, OUT1, OUT2, PMODE, SLP, VIN; removed none
- sheet LSM6DSO ports: added none; removed CS, INT1, INT2, OCS Aux, SCx, SDO, SDO Aux, SDx, VDD
- company: (none) -> Cal Poly
- moved on the sheet: J1, U1
