File: Nemesis/Nemesis.kicad_pcb (KiCad board)
At the start: 2 copper layers, 54 parts, among them Q1 Q_PMOS, Q2 Q_PMOS, U1 NODEMCU-32S, U2 DRV8874PWPR, U3 LSM6DSO, U4 DRV8874PWPR

Commit message: Add files via upload
Parts:
- S13V20F5: footprint TerminalBlock_Phoenix:TerminalBlock_Phoenix_MKDS-1,5-3-5.08_1x03_P5.08mm_Horizontal -> Connector_PinHeader_2.54mm:PinHeader_1x03_P2.54mm_Vertical
- moved S13V20F5 51.3 mm to (109.9, 40.0), turned to 90 degrees
- renumbered R19 to R18, R20 to R19
Connections:
- net /DRV8874/CS renamed /DRV8874-1/CS
- net /DRV8874/FLT renamed /DRV8874-1/FLT
- net /DRV8874/IMODE renamed /DRV8874-1/IMODE
- net /DRV8874/OUT1 renamed /DRV8874-1/OUT1
- net /DRV8874/OUT2 renamed /DRV8874-1/OUT2
- net /DRV8874/VM renamed /DRV8874-1/VM
- net /DRV8874/VREF renamed /DRV8874-1/VREF
- net /DRV8875/CS renamed /DRV8874-2/CS
- net /DRV8875/FLT renamed /DRV8874-2/FLT
- net /DRV8875/IMODE renamed /DRV8874-2/IMODE
- net /DRV8875/OUT1 renamed /DRV8874-2/OUT1
- net /DRV8875/OUT2 renamed /DRV8874-2/OUT2
- net /DRV8875/VM renamed /DRV8874-2/VM
- net /DRV8875/VREF renamed /DRV8874-2/VREF
